Commit message: Separate unit test out (one .cpp file per class), AnalyticalSolver handles both Yaml/URDF for getting link lengths (and this is configured in Yaml file). Add Placeholder PinocchioSolver tests that fail

File: include/planar_arm_kinematics/config/urdf/planar_arm.urdf (robot description, URDF)
Before this commit: robot planar_arm, 6 links, 5 joints
Joints:
- joint joint_1: origin xyz=0.0 0.0 156.92000e-3 rpy=0.0 0.0 0.0 -> xyz=0.0 0.0 20.0e-3 rpy=0.0 0.0 0.0
- joint joint_2: origin xyz=0.0 0.0 67.96380e-3 rpy=0.0 0.0 0.0 -> xyz=300.0e-3 0.0 0.0 rpy=0.0 0.0 0.0
- joint joint_3: origin xyz=150.0e-3 0.0 0.0 rpy=0.0 0.0 0.0 -> xyz=300.0e-3 0.0 0.0 rpy=0.0 0.0 0.0

Commit message: Fix URDF bug: (0 0 1) vs. (0 -1 0) joint axis issue

File: include/planar_arm_kinematics/config/urdf/planar_arm.urdf (robot description, URDF)
Before this commit: robot planar_arm, 6 links, 5 joints
Joints:
- joint joint_2: axis 0 -1 0 -> 0 0 1
- joint joint_3: axis 0 -1 0 -> 0 0 1
